File: hardware/NfcCarrierBoard/NfcCarrierBoard.kicad_sch (KiCad schematic)
At the start: 51 parts, among them J1 Barrel_Jack, J2 Conn_01x03, J3 JST SH 4, J4 Grove, J5 Conn_01x03, J6 UART, J7 Grove UART, Q1 NMOS, Q2 NMOS, SW1 RESET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

Commit message: Add jumper to bypass audio pot
Parts:
- added JP4: SolderJumper_2_Open, Jumper:SolderJumper-2_P1.3mm_Open_RoundedPad1.0x1.5mm, symbol Jumper:SolderJumper_2_Open
- RV1: footprint (none) -> Potentiometer_THT:Potentiometer_Runtron_RM-065_Vertical
Connections:
- net at BZ1.1 (+), D2.1 (K), RV1.3: now also JP4.1 (A)
- net at C1.1, R3.1, RV1.2: now also JP4.2 (B)
Other:
- moved on the sheet: RV1
Changed lines of the file:
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@@
 	)
 	(junction
+		(at 54.61 148.59)
+		(diameter 0)
+		(color 0 0 0 0)
+	)
+	(junction
+		(at 48.26 156.21)
+		(diameter 0)
+		(color 0 0 0 0)
+	)
+	(junction
 		(at 215.9 35.56)
 		(diameter 0)
@@
 	)
 	(junction
-		(at 52.07 156.21)
+		(at 54.61 156.21)
 		(diameter 0)
 		(color 0 0 0 0)
@@
 	)
 	(no_connect
-		(at 52.07 144.78)
+		(at 48.26 144.78)
 	)
 	(no_connect
@@
 	(wire
 		(pts
+			(xy 52.07 148.59) (xy 54.61 148.59)
+		)
+		(stroke
+			(width 0)
+			(type default)
+		)
+	)
+	(wire
+		(pts
 			(xy 31.75 71.12) (xy 38.1 71.12)
 		)
@@
 	(wire
 		(pts
-			(xy 55.88 156.21) (xy 52.07 156.21)
-		)
-		(stroke
-			(width 0)
-			(type default)
-		)
-	)
-	(wire
-		(pts
 			(xy 234.95 25.4) (xy 234.95 22.86)
 		)
@@
 	(wire
 		(pts
+			(xy 48.26 156.21) (xy 54.61 156.21)
+		)
+		(stroke
+			(width 0)
+			(type default)
+		)
+	)
+	(wire
+		(pts
 			(xy 262.89 68.58) (xy 266.7 68.58)
 		)
@@
 	(wire
 		(pts
-			(xy 52.07 152.4) (xy 52.07 156.21)
-		)
-		(stroke
-			(width 0)
-			(type default)
-		)
-	)
-	(wire
-		(pts
-			(xy 55.88 148.59) (xy 67.31 148.59)
+			(xy 48.26 152.4) (xy 48.26 156.21)
 		)
 		(stroke
@@
 	(wire
 		(pts
-			(xy 46.99 156.21) (xy 52.07 156.21)
+			(xy 46.99 156.21) (xy 48.26 156.21)
 		)
 		(stroke
@@
 	(wire
 		(pts
+			(xy 54.61 148.59) (xy 67.31 148.59)
+		)
+		(stroke
+			(width 0)
+			(type default)
+		)
+	)
+	(wire
+		(pts
 			(xy 29.21 93.98) (xy 29.21 96.52)
 		)
@@
 	(wire
 		(pts
+			(xy 54.61 156.21) (xy 55.88 156.21)
+		)
+		(stroke
+			(width 0)
+			(type default)
+		)
+	)
+	(wire
+		(pts
 			(xy 232.41 81.28) (xy 237.49 81.28)
 		)
@@
 	)
 	(symbol
+		(lib_id "Jumper:SolderJumper_2_Open")
+		(at 54.61 152.4 90)
+		(unit 1)
+		(exclude_from_sim yes)
+		(in_bom no)
+		(on_board yes)
+		(dnp no)
+		(fields_autoplaced yes)
+		(property "Reference" "JP4"
+			(at 57.15 152.3999 90)
+			(effects
+				(font
+					(size 1.27 1.27)
+				)
+				(justify right)
+			)
+		)
+		(property "Value" "SolderJumper_2_Open"
+			(at 57.15 153.6699 90)
+			(effects
+				(font
+					(size 1.27 1.27)
+				)
+				(justify right)
+				(hide yes)
+			)
+		)
+		(property "Footprint" "Jumper:SolderJumper-2_P1.3mm_Open_RoundedPad1.0x1.5mm"
+			(at 54.61 152.4 0)
+			(effects
+				(font
+					(size 1.27 1.27)
+				)
+				(hide yes)
+			)
+		)
+		(property "Datasheet" "~"
+			(at 54.61 152.4 0)
+			(effects
+				(font
+					(size 1.27 1.27)
+				)
+				(hide yes)
+			)
+		)
+		(property "Description" "Solder Jumper, 2-pole, open"
+			(at 54.61 152.4 0)
+			(effects
+				(font
+					(size 1.27 1.27)
+				)
+				(hide yes)
+			)
+		)
+		(pin "2"
+		)
+		(pin "1"
+		)
+		(instances
+			(project ""
+				(path "/766243a7-ad3d-48cd-bfed-d2ecca850827"
+					(reference "JP4")
+					(unit 1)
+				)
+			)
+		)
+	)
+	(symbol
 		(lib_id "power:GND")
 		(at 29.21 96.52 0)
@@
 	(symbol
 		(lib_id "Device:R_Potentiometer_Trim")
-		(at 52.07 148.59 0)
+		(at 48.26 148.59 0)
 		(unit 1)
 		(exclude_from_sim no)
@@
 		(fields_autoplaced yes)
 		(property "Reference" "RV1"
-			(at 49.53 147.3199 0)
+			(at 45.72 147.3199 0)
 			(effects
 				(font
@@
 		)
 		(property "Value" "R_Potentiometer_Trim"
-			(at 49.53 149.8599 0)
+			(at 45.72 149.8599 0)
 			(effects
 				(font
@@
 			)
 		)
-		(property "Footprint" ""
-			(at 52.07 148.59 0)
+		(property "Footprint" "Potentiometer_THT:Potentiometer_Runtron_RM-065_Vertical"
+			(at 48.26 148.59 0)
 			(effects
 				(font
@@
 		)
 		(property "Datasheet" "~"
-			(at 52.07 148.59 0)
+			(at 48.26 148.59 0)
 			(effects
 				(font
@@
 		)
 		(property "Description" "Trim-potentiometer"
-			(at 52.07 148.59 0)
+			(at 48.26 148.59 0)
 			(effects
 				(font

Commit message: Add mounting holes Add OSHW logo Change Ethernet footprint
Parts:
- added H1, H2, H3, H4: MountingHole, MountingHole:MountingHole_3.2mm_M3, symbol Mechanical:MountingHole
- A2: value ~ -> Ethernet FeatherWing; footprint Module:Adafruit_Feather -> FootprintLibrary:Adafruit_Ethernet_FeatherWing

Commit message: Add custom footprint for 0603 0805 1206 jellybean parts
Parts:
- C1, C10, C2, C3, C4, C5, C6, C7, C8, C9: footprint Capacitor_SMD:C_0805_2012Metric_Pad1.18x1.45mm_HandSolder -> FootprintLibrary:SMD_HANDSOLDER_UNIVERSAL_0603_0805_1206
- D1, D2: footprint Diode_SMD:D_SMA-SMB_Universal_Handsoldering -> FootprintLibrary:SMD_HANDSOLDER_UNIVERSAL_0603_0805_1206
- R1, R2, R3, R4, R5, R6, R7, R8: footprint Resistor_SMD:R_0805_2012Metric_Pad1.20x1.40mm_HandSolder -> FootprintLibrary:SMD_HANDSOLDER_UNIVERSAL_0603_0805_1206
Changed lines of the file:
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@@
 			)
 		)
-		(property "Footprint" "Resistor_SMD:R_0805_2012Metric_Pad1.20x1.40mm_HandSolder"
+		(property "Footprint" "FootprintLibrary:SMD_HANDSOLDER_UNIVERSAL_0603_0805_1206"
 			(at 42.418 179.07 90)
 			(effects
@@
 			)
 		)
-		(property "Footprint" "Resistor_SMD:R_0805_2012Metric_Pad1.20x1.40mm_HandSolder"
+		(property "Footprint" "FootprintLibrary:SMD_HANDSOLDER_UNIVERSAL_0603_0805_1206"
 			(at 157.988 154.94 90)
 			(effects
@@
 			)
 		)
-		(property "Footprint" "Capacitor_SMD:C_0805_2012Metric_Pad1.18x1.45mm_HandSolder"
+		(property "Footprint" "FootprintLibrary:SMD_HANDSOLDER_UNIVERSAL_0603_0805_1206"
 			(at 98.7552 127 0)
 			(effects
@@
 			)
 		)
-		(property "Footprint" "Diode_SMD:D_SMA-SMB_Universal_Handsoldering"
+		(property "Footprint" "FootprintLibrary:SMD_HANDSOLDER_UNIVERSAL_0603_0805_1206"
 			(at 129.54 119.38 0)
 			(effects
@@
 			)
 		)
-		(property "Footprint" "Capacitor_SMD:C_0805_2012Metric_Pad1.18x1.45mm_HandSolder"
+		(property "Footprint" "FootprintLibrary:SMD_HANDSOLDER_UNIVERSAL_0603_0805_1206"
 			(at 207.9752 78.74 0)
 			(effects
@@
 			)
 		)
-		(property "Footprint" "Resistor_SMD:R_0805_2012Metric_Pad1.20x1.40mm_HandSolder"
+		(property "Footprint" "FootprintLibrary:SMD_HANDSOLDER_UNIVERSAL_0603_0805_1206"
 			(at 172.212 71.12 90)
 			(effects
@@
 			)
 		)
-		(property "Footprint" "Capacitor_SMD:C_0805_2012Metric_Pad1.18x1.45mm_HandSolder"
+		(property "Footprint" "FootprintLibrary:SMD_HANDSOLDER_UNIVERSAL_0603_0805_1206"
 			(at 68.2752 158.75 0)
 			(effects
@@
 			)
 		)
-		(property "Footprint" "Resistor_SMD:R_0805_2012Metric_Pad1.20x1.40mm_HandSolder"
+		(property "Footprint" "FootprintLibrary:SMD_HANDSOLDER_UNIVERSAL_0603_0805_1206"
 			(at 217.678 30.48 90)
 			(effects
@@
 			)
 		)
-		(property "Footprint" "Diode_SMD:D_SMA-SMB_Universal_Handsoldering"
+		(property "Footprint" "FootprintLibrary:SMD_HANDSOLDER_UNIVERSAL_0603_0805_1206"
 			(at 46.99 160.02 0)
 			(effects
@@
 			)
 		)
-		(property "Footprint" "Capacitor_SMD:C_0805_2012Metric_Pad1.18x1.45mm_HandSolder"
+		(property "Footprint" "FootprintLibrary:SMD_HANDSOLDER_UNIVERSAL_0603_0805_1206"
 			(at 139.3952 181.61 0)
 			(effects
@@
 			)
 		)
-		(property "Footprint" "Capacitor_SMD:C_0805_2012Metric_Pad1.18x1.45mm_HandSolder"
+		(property "Footprint" "FootprintLibrary:SMD_HANDSOLDER_UNIVERSAL_0603_0805_1206"
 			(at 275.8948 43.18 0)
 			(effects
@@
 			)
 		)
-		(property "Footprint" "Resistor_SMD:R_0805_2012Metric_Pad1.20x1.40mm_HandSolder"
+		(property "Footprint" "FootprintLibrary:SMD_HANDSOLDER_UNIVERSAL_0603_0805_1206"
 			(at 227.838 30.48 90)
 			(effects
@@
 			)
 		)
-		(property "Footprint" "Capacitor_SMD:C_0805_2012Metric_Pad1.18x1.45mm_HandSolder"
+		(property "Footprint" "FootprintLibrary:SMD_HANDSOLDER_UNIVERSAL_0603_0805_1206"
 			(at 70.8152 96.52 0)
 			(effects
@@
 			)
 		)
-		(property "Footprint" "Resistor_SMD:R_0805_2012Metric_Pad1.20x1.40mm_HandSolder"
+		(property "Footprint" "FootprintLibrary:SMD_HANDSOLDER_UNIVERSAL_0603_0805_1206"
 			(at 33.02 172.212 90)
 			(effects
@@
 			)
 		)
-		(property "Footprint" "Resistor_SMD:R_0805_2012Metric_Pad1.20x1.40mm_HandSolder"
+		(property "Footprint" "FootprintLibrary:SMD_HANDSOLDER_UNIVERSAL_0603_0805_1206"
 			(at 73.66 146.812 90)
 			(effects
@@
 			)
 		)
-		(property "Footprint" "Capacitor_SMD:C_0805_2012Metric_Pad1.18x1.45mm_HandSolder"
+		(property "Footprint" "FootprintLibrary:SMD_HANDSOLDER_UNIVERSAL_0603_0805_1206"
 			(at 147.0152 82.55 0)
 			(effects
@@
 			)
 		)
-		(property "Footprint" "Resistor_SMD:R_0805_2012Metric_Pad1.20x1.40mm_HandSolder"
+		(property "Footprint" "FootprintLibrary:SMD_HANDSOLDER_UNIVERSAL_0603_0805_1206"
 			(at 139.192 154.94 90)
 			(effects
@@
 			)
 		)
-		(property "Footprint" "Capacitor_SMD:C_0805_2012Metric_Pad1.18x1.45mm_HandSolder"
+		(property "Footprint" "FootprintLibrary:SMD_HANDSOLDER_UNIVERSAL_0603_0805_1206"
 			(at 83.5152 96.52 0)
 			(effects
@@
 			)
 		)
-		(property "Footprint" "Capacitor_SMD:C_0805_2012Metric_Pad1.18x1.45mm_HandSolder"
+		(property "Footprint" "FootprintLibrary:SMD_HANDSOLDER_UNIVERSAL_0603_0805_1206"
 			(at 199.0852 149.86 0)
 			(effects
@@
 			)
 		)
-		(property "Footprint" "Capacitor_SMD:C_0805_2012Metric_Pad1.18x1.45mm_HandSolder"
+		(property "Footprint" "FootprintLibrary:SMD_HANDSOLDER_UNIVERSAL_0603_0805_1206"
 			(at 80.9752 158.75 0)
 			(effects

Commit message: Add reset switch footprint and 3d model
Parts:
- SW1: footprint (none) -> FootprintLibrary:SW_TS11-674-105-BK-260-RA-D; symbol Switch:SW_Push -> Switch:SW_Push_Shielded
Connections:
- net GND: now also SW1.SH (B)
Changed lines of the file:
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@@
 	)
 	(junction
+		(at 205.74 152.4)
+		(diameter 0)
+		(color 0 0 0 0)
+	)
+	(junction
 		(at 135.89 119.38)
 		(diameter 0)
@@
 	(wire
 		(pts
-			(xy 198.12 152.4) (xy 213.36 152.4)
+			(xy 198.12 152.4) (xy 205.74 152.4)
 		)
 		(stroke
@@
 	(wire
 		(pts
+			(xy 205.74 143.51) (xy 205.74 152.4)
+		)
+		(stroke
+			(width 0)
+			(type default)
+		)
+	)
+	(wire
+		(pts
 			(xy 140.97 124.46) (xy 140.97 127)
 		)
@@
 	(wire
 		(pts
+			(xy 205.74 152.4) (xy 213.36 152.4)
+		)
+		(stroke
+			(width 0)
+			(type default)
+		)
+	)
+	(wire
+		(pts
 			(xy 40.64 182.88) (xy 40.64 184.15)
 		)
@@
 	)
 	(symbol
-		(lib_id "Switch:SW_Push")
+		(lib_id "Switch:SW_Push_Shielded")
 		(at 205.74 139.7 0)
 		(unit 1)
@@
 			)
 		)
-		(property "Footprint" ""
+		(property "Footprint" "FootprintLibrary:SW_TS11-674-105-BK-260-RA-D"
 			(at 205.74 134.62 0)
 			(effects
@@
 			)
 		)
-		(property "Description" "Push button switch, generic, two pins"
+		(property "Description" "Generic push-button switch, two contact pins and shield pin(s)"
 			(at 205.74 139.7 0)
 			(effects
@@
 		(pin "2"
 		)
+		(pin "SH"
+		)
 		(instances
 			(project ""
@@
 		(lib_id "Device:C")
 		(at 198.12 146.05 0)
+		(mirror y)
 		(unit 1)
 		(exclude_from_sim no)
@@
 		(on_board yes)
 		(dnp no)
-		(fields_autoplaced yes)
 		(property "Reference" "C3"
-			(at 201.93 144.7799 0)
+			(at 194.31 144.7799 0)
 			(effects
 				(font
@@
 		)
 		(property "Value" "0.1µF"
-			(at 201.93 147.3199 0)
+			(at 194.31 147.3199 0)
 			(effects
 				(font
@@
 		)
 		(property "Footprint" "FootprintLibrary:SMD_HANDSOLDER_UNIVERSAL_0603_0805_1206"
-			(at 199.0852 149.86 0)
+			(at 197.1548 149.86 0)
 			(effects
 				(font

Commit message: Update switch footprint to match KiCAD pin naming
Parts:
- SW1: DigiKey PN (none) -> 2223-TS11-674-105-BK-260-RA-D-ND; MPN (none) -> TS11-674-105-BK-260-RA-D
Changed lines of the file:
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@@
+			)
+		)
+		(property "MPN" "TS11-674-105-BK-260-RA-D"
+			(at 205.74 139.7 0)
+			(effects
+				(font
+					(size 1.27 1.27)
+				)
+				(hide yes)
+			)
+		)
+		(property "DigiKey PN" "2223-TS11-674-105-BK-260-RA-D-ND"
+			(at 205.74 139.7 0)
+			(effects
+				(font
+					(size 1.27 1.27)
+				)
+				(hide yes)
 			)
 		)

Commit message: Begin work on PCB layout
Parts:
- TP1, TP2: footprint TestPoint:TestPoint_THTPad_D2.0mm_Drill1.0mm -> TestPoint:TestPoint_Pad_D2.0mm
Connections:
- net +12V Input: now reaches D1.2 (A), J1.1
Changed lines of the file:
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@@
 		)
 	)
+	(global_label "+12V Input"
+		(shape passive)
+		(at 124.46 119.38 90)
+		(fields_autoplaced yes)
+		(effects
+			(font
+				(size 1.27 1.27)
+			)
+			(justify left)
+		)
+		(property "Intersheetrefs" "${INTERSHEET_REFS}"
+			(at 124.46 106.681 90)
+			(effects
+				(font
+					(size 1.27 1.27)
+				)
+				(justify left)
+				(hide yes)
+			)
+		)
+	)
 	(global_label "TX"
 		(shape input)
@@
 			)
 		)
-		(property "Footprint" "TestPoint:TestPoint_THTPad_D2.0mm_Drill1.0mm"
+		(property "Footprint" "TestPoint:TestPoint_Pad_D2.0mm"
 			(at 267.97 97.79 0)
 			(effects
@@
 			)
 		)
-		(property "Footprint" "TestPoint:TestPoint_THTPad_D2.0mm_Drill1.0mm"
+		(property "Footprint" "TestPoint:TestPoint_Pad_D2.0mm"
 			(at 267.97 101.6 0)
 			(effects
