File: hardware/NfcCarrierBoard/NfcCarrierBoard.kicad_sch (KiCad schematic)
At the start: 58 parts, among them J1 Barrel_Jack, J2 Conn_01x03, J3 JST SH 4, J4 Grove, J5 Conn_01x03, J6 UART, J7 Grove UART, Q1 NMOS, Q2 NMOS, SW1 RESET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

Commit message: Fix BOM output
Parts:
- HS1, TP1, TP2, TP4: now left out of the parts list
Changed lines of the file:
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@@
 		(unit 1)
 		(exclude_from_sim no)
-		(in_bom yes)
+		(in_bom no)
 		(on_board yes)
 		(dnp no)
@@
 		(unit 1)
 		(exclude_from_sim no)
-		(in_bom yes)
+		(in_bom no)
 		(on_board yes)
 		(dnp no)
@@
 		(unit 1)
 		(exclude_from_sim no)
-		(in_bom yes)
+		(in_bom no)
 		(on_board yes)
 		(dnp no)
@@
 		(unit 1)
 		(exclude_from_sim no)
-		(in_bom yes)
+		(in_bom no)
 		(on_board yes)
 		(dnp no)

Commit message: Fix #42
Parts:
- A2: footprint FootprintLibrary:Adafruit_Ethernet_FeatherWing -> Module:Adafruit_Feather
Connections:
- net SCK: now also A2.11 (SCK); no longer A2.13 (SCK)
- net SDI: now also A2.13 (SDI); no longer A2.12 (SDI)
- net SDO: now also A2.12 (SDO); no longer A2.11 (SDO)
Changed lines of the file:
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@@
 	)
 	(symbol
-		(lib_name "Silicognition_PoE_FeatherWing_1")
 		(lib_id "SymbolLibrary:Silicognition_PoE_FeatherWing")
 		(at 250.19 77.47 0)
@@
 			)
 		)
-		(property "Footprint" "FootprintLibrary:Adafruit_Ethernet_FeatherWing"
+		(property "Footprint" "Module:Adafruit_Feather"
 			(at 250.444 94.742 0)
 			(effects
