File: hardware/NfcCarrierBoard/NfcCarrierBoard.kicad_pcb (KiCad board)
At the start: 2 copper layers, 80 x 100 mm, 50 parts, among them J1 Barrel_Jack, J2 Conn_01x03, J3 JST SH 4, J4 Grove, J5 Conn_01x03, J6 UART, J7 Grove UART, Q1 NMOS, Q2 NMOS, SW1 RESET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

Commit message: Import updated BOM from schematic to PCB
Parts:
- R1: value ~10kΩ -> 10kΩ

Commit message: Fix #42
Parts:
- A2: footprint FootprintLibrary:Adafruit_Ethernet_FeatherWing -> Module:Adafruit_Feather
Connections:
- A2 pad 11: SDO -> SCK
- A2 pad 12: SDI -> SDO
- A2 pad 13: SCK -> SDI
Routing:
- net SCK: track 18.5 -> 7.15 mm
- net SDO: track 10.3 -> 17.5 mm
- net SDI: track 18.6 -> 25.0 mm
- net GND: vias 57 -> 59
